Commit message: Add files via upload

File: leg.urdf.xacro (robot description, xacro)
@@ -22,7 +22,8 @@
             <xacro:property name="upper_leg_to_lower_leg" value="-${upper_leg_to_lower_leg_distance}" />
         </xacro:if>
-        <xacro:property name="hip_mesh_path" value="package://robot_sim_description/meshes/${leg}_hip.stl" />
-        <xacro:property name="upper_leg_mesh_path" value="package://robot_sim_description/meshes/${leg}_upper_leg.stl" />
-        <xacro:property name="lower_leg_mesh_path" value="package://robot_sim_description/meshes/${leg}_lower_leg.stl" />
+        <xacro:property name="hip_mesh_path" value="package://robot_sim_description/meshes/${leg}_hipp.stl" />
+        <xacro:property name="upper_leg_mesh_path" value="package://robot_sim_description/meshes/${leg}_up.stl" />
+        <xacro:property name="lower_leg_mesh_path" value="package://robot_sim_description/meshes/${leg}_low.stl" />
+        <xacro:property name="foot_mesh_path" value="package://robot_sim_description/meshes/${leg}_foot.stl" />
         <link name="${leg}_hip_link">
             <inertial>

File: robot_sim.urdf (robot description, URDF)
Before this commit: robot mini-pupper, 18 links, 17 joints
Links:
- removed link lf_hip_link
- removed link lf_lower_leg_link
- removed link lf_upper_leg_link
- removed link lh_hip_link
- removed link lh_lower_leg_link
- removed link lh_upper_leg_link
- removed link rf_hip_link
- removed link rf_lower_leg_link
- removed link rf_upper_leg_link
- removed link rh_hip_link
- removed link rh_lower_leg_link
- removed link rh_upper_leg_link
- added link lf_hipp_link, mass 0.7; collision mesh filename=package://robot_sim_description/meshes/lf_hipp.stl scale=0.001 0.001 0.001; visual mesh filename=package://robot_sim_description/meshes/lf_hipp.stl scale=0.001 0.001 0.001
- added link lf_low_link, mass 0.2; collision mesh filename=package://robot_sim_description/meshes/lf_low.stl scale=0.001 0.001 0.001; visual mesh filename=package://robot_sim_description/meshes/lf_low.stl scale=0.001 0.001 0.001
- added link lf_up_link, mass 0.2; collision mesh filename=package://robot_sim_description/meshes/lf_up.stl scale=0.001 0.001 0.001; visual mesh filename=package://robot_sim_description/meshes/lf_up.stl scale=0.001 0.001 0.001
- added link lh_hipp_link, mass 0.7; collision mesh filename=package://robot_sim_description/meshes/lh_hipp.stl scale=0.001 0.001 0.001; visual mesh filename=package://robot_sim_description/meshes/lh_hipp.stl scale=0.001 0.001 0.001
- added link lh_low_link, mass 0.2; collision mesh filename=package://robot_sim_description/meshes/lh_low.stl scale=0.001 0.001 0.001; visual mesh filename=package://robot_sim_description/meshes/lh_low.stl scale=0.001 0.001 0.001
- added link lh_up_link, mass 0.2; collision mesh filename=package://robot_sim_description/meshes/lh_up.stl scale=0.001 0.001 0.001; visual mesh filename=package://robot_sim_description/meshes/lh_up.stl scale=0.001 0.001 0.001
- added link rf_hipp_link, mass 0.7; collision mesh filename=package://robot_sim_description/meshes/rf_hippp.stl scale=0.001 0.001 0.001; visual mesh filename=package://robot_sim_description/meshes/rf_hipp.stl scale=0.001 0.001 0.001
- added link rf_low_link, mass 0.2; collision mesh filename=package://robot_sim_description/meshes/rf_low.stl scale=0.001 0.001 0.001; visual mesh filename=package://robot_sim_description/meshes/rf_low.stl scale=0.001 0.001 0.001
- added link rf_up_link, mass 0.2; collision mesh filename=package://robot_sim_description/meshes/rf_up.stl scale=0.001 0.001 0.001; visual mesh filename=package://robot_sim_description/meshes/rf_up.stl scale=0.001 0.001 0.001
- added link rh_hipp_link, mass 0.7; collision mesh filename=package://robot_sim_description/meshes/rh_hipp.stl scale=0.001 0.001 0.001; visual mesh filename=package://robot_sim_description/meshes/rh_hipp.stl scale=0.001 0.001 0.001
- added link rh_low_link, mass 0.2; collision mesh filename=package://robot_sim_description/meshes/rh_low.stl scale=0.001 0.001 0.001; visual mesh filename=package://robot_sim_description/meshes/rh_low.stl scale=0.001 0.001 0.001
- added link rh_up_link, mass 0.2; collision mesh filename=package://robot_sim_description/meshes/rh_up.stl scale=0.001 0.001 0.001; visual mesh filename=package://robot_sim_description/meshes/rh_up.stl scale=0.001 0.001 0.001
- link lf_foot_link: geometry collision sphere radius=0.02; visual mesh filename=package://robot_sim_description/meshes/lf_foot.stl scale=0.001 0.001 0.001
- link lh_foot_link: geometry collision sphere radius=0.02; visual mesh filename=package://robot_sim_description/meshes/lh_foot.stl scale=0.001 0.001 0.001
- link rf_foot_link: geometry collision sphere radius=0.02; visual mesh filename=package://robot_sim_description/meshes/rf_foot.stl scale=0.001 0.001 0.001
- link rh_foot_link: geometry collision sphere radius=0.02; visual mesh filename=package://robot_sim_description/meshes/rh_foot.stl scale=0.001 0.001 0.001
Joints:
- removed joint lf_hip_joint
- removed joint lf_lower_leg_joint
- removed joint lf_upper_leg_joint
- removed joint lh_hip_joint
- removed joint lh_lower_leg_joint
- removed joint lh_upper_leg_joint
- removed joint rf_hip_joint
- removed joint rf_lower_leg_joint
- removed joint rf_upper_leg_joint
- removed joint rh_hip_joint
- removed joint rh_lower_leg_joint
- removed joint rh_upper_leg_joint
- added joint lf_hipp_joint: type revolute, parent base_link, child lf_hipp_link, origin xyz=0.04469 0.04937 0.01767 rpy=0 0 0, axis 1 0 0, limit lower=-3.14 upper=3.14 effort=5 velocity=2.5
- added joint lf_low_joint: type revolute, parent lf_up_link, child lf_low_link, origin xyz=0 0.0075 -0.0653 rpy=0 0 0, axis 0 1 0, limit lower=-3.14 upper=3.14 effort=5 velocity=2.5
- added joint lf_up_joint: type revolute, parent lf_hipp_link, child lf_up_link, origin xyz=0 0.0266 0 rpy=0 0 0, axis 0 1 0, limit lower=-3.14 upper=3.14 effort=5 velocity=2.5
- added joint lh_hipp_joint: type revolute, parent base_link, child lh_hipp_link, origin xyz=-0.04640 0.04937 0.01767 rpy=0 0 0, axis 1 0 0, limit lower=-3.14 upper=3.14 effort=5 velocity=2.5
- added joint lh_low_joint: type revolute, parent lh_up_link, child lh_low_link, origin xyz=0 0.0075 -0.0653 rpy=0 0 0, axis 0 1 0, limit lower=-3.14 upper=3.14 effort=5 velocity=2.5
- added joint lh_up_joint: type revolute, parent lh_hipp_link, child lh_up_link, origin xyz=0 0.0266 0 rpy=0 0 0, axis 0 1 0, limit lower=-3.14 upper=3.14 effort=5 velocity=2.5
- added joint rf_hipp_joint: type revolute, parent base_link, child rf_hipp_link, origin xyz=0.04469 -0.04937 0.01767 rpy=0 0 0, axis 1 0 0, limit lower=-3.14 upper=3.14 effort=5 velocity=2.5
- added joint rf_low_joint: type revolute, parent rf_up_link, child rf_low_link, origin xyz=0 -0.0075 -0.0653 rpy=0 0 0, axis 0 1 0, limit lower=-3.14 upper=3.14 effort=5 velocity=2.5
- added joint rf_up_joint: type revolute, parent rf_hipp_link, child rf_up_link, origin xyz=0 -0.0266 0 rpy=0 0 0, axis 0 1 0, limit lower=-3.14 upper=3.14 effort=5 velocity=2.5
- added joint rh_hipp_joint: type revolute, parent base_link, child rh_hipp_link, origin xyz=-0.04640 -0.04937 0.01767 rpy=0 0 0, axis 1 0 0, limit lower=-3.14 upper=3.14 effort=5 velocity=2.5
- added joint rh_low_joint: type revolute, parent rh_up_link, child rh_low_link, origin xyz=0 -0.0075 -0.0653 rpy=0 0 0, axis 0 1 0, limit lower=-3.14 upper=3.14 effort=5 velocity=2.5
- added joint rh_up_joint: type revolute, parent rh_hipp_link, child rh_up_link, origin xyz=0 -0.0266 0 rpy=0 0 0, axis 0 1 0, limit lower=-3.14 upper=3.14 effort=5 velocity=2.5
- joint lf_foot_joint: parent lf_lower_leg_link -> lf_low_link
- joint lh_foot_joint: parent lh_lower_leg_link -> lh_low_link
- joint rf_foot_joint: parent rf_lower_leg_link -> rf_low_link
- joint rh_foot_joint: parent rh_lower_leg_link -> rh_low_link
